File: Section A - Title A.kicad_sch (KiCad schematic)
At the start: 0 parts

Commit message: Backup before adding module net labels
Parts:
- added TP1: TestPoint_Probe, TestPoint:TestPoint_Pad_D1.0mm, symbol Connector:TestPoint_Probe
- added U1: ME54BS13_V1.0, ME54BS13_V1.0, symbol minew:ME54BS13_V1.0
Connections:
- new net +3V3: U1.19 (VCC)
- new net GND: U1.1 (GND), U1.10 (GND), U1.11 (GND), U1.20 (GND), U1.3 (GND), U1.D0 (GND), U1.E0 (GND), U1.F0 (GND)
- new net RST_NRF54: U1.4 (nRESET)
- new net SWDCLK_NRF54: TP1.1, U1.6 (SWDCLK)
- new net SWDIO_NRF54: U1.5 (SWDIO)
- no-connect marks 0 -> 1
