File: palroc_one_pcb.kicad_pcb (KiCad board)
At the start: 6 copper layers, 0 parts

Commit message: Backup before adding module net labels
Parts:
- added U1: ME54BS13_V1.0, minew:ME54BS13_V1.0, F.Cu at (142.5, 96.3)
