File: Misc.kicad_sch (KiCad schematic)
At the start: 56 parts, among them J2 Screw_Terminal_01x02, Q3 SSM6N56FE,LM, Q4 SSM6N56FE,LM, Q5 SSM6N56FE,LM, SW1 ZX-QC66-8.5TP, SW2 ZX-QC66-8.5TP, SW3 ZX-QC66-8.5TP, SW4 ZX-QC66-8.5TP, U11 LIS2DW12TR, U7 MAX98357AETE+T, U9 W25Q128JVPIQTR

Commit message: Update footprint 3D models, add through-hole connector, and refine PCB layout
Refreshes 3D shapes/step models across several component libraries,
adds a new XY308 2.54mm through-hole connector footprint, and updates
PCB placement/routing and CI workflow.

Co-Authored-By: Claude Sonnet 5 <noreply@anthropic.com>
Parts:
- J2: footprint TerminalBlock:TerminalBlock_Xinya_XY308-2.54-2P_1x02_P2.54mm_Horizontal -> PALROC_Connectorss:CONN-TH_XY308-2.54-2P
Changed lines of the file:
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@@
 			)
 		)
-		(property "Footprint" "TerminalBlock:TerminalBlock_Xinya_XY308-2.54-2P_1x02_P2.54mm_Horizontal"
+		(property "Footprint" "PALROC_Connectorss:CONN-TH_XY308-2.54-2P"
 			(at 389.89 58.42 0)
 			(effects
@@
 					(size 1.27 1.27)
 				)
-				(hide yes)
 			)
 		)
